File: kicad/digital_probe/digital_probe.kicad_pcb (KiCad board)
At the start: 2 copper layers, 45.5 x 72.4 mm, 33 parts, among them J1 Conn_02x08_Odd_Even, J2 Conn_02x08_Odd_Even, J3 Conn_02x25_Odd_Even, J4 D8-15 Vref, J5 D0-7 Vref, U1 MC33375ST

Commit message: изменено:      kicad/digital_probe/digital_probe-cache.lib 	изменено:      kicad/digital_probe/digital_probe.kicad_pcb 	изменено:      kicad/digital_probe/digital_probe.kicad_pcb-bak 	изменено:      kicad/digital_probe/digital_probe.sch 	изменено:      kicad/digital_probe/digital_probe.sch-bak
Parts:
- moved C3 34.6 mm to (55.1, 94.3)
- moved C4 34.6 mm to (54.5, 85.9)
- moved C5 34.6 mm to (55.0, 99.1)
- moved C7 34.6 mm to (59.8, 89.5)
- moved J1 34.6 mm to (40.6, 88.4)
- moved J2 34.6 mm to (40.6, 116.6)
- moved R1 34.6 mm to (50.5, 84.2)
- moved R8 34.6 mm to (43.6, 75.7)
- moved U1 34.6 mm to (59.8, 83.6)
- moved C1 34.6 mm to (55.1, 88.6)
- moved C2 34.6 mm to (55.2, 92.1)
- moved D1 34.6 mm to (51.3, 82.5)
- moved D2 34.6 mm to (56.2, 92.1)
- moved J3 34.6 mm to (72.0, 56.4)
- moved J4 34.6 mm to (67.2, 62.6)
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Routing:
- net +3V3: track 37.3 -> 42.2 mm

Commit message: изменено:      kicad/digital_probe/digital_probe-cache.lib 	изменено:      kicad/digital_probe/digital_probe.kicad_pcb 	изменено:      kicad/digital_probe/digital_probe.kicad_pcb-bak 	изменено:      kicad/digital_probe/digital_probe.sch 	изменено:      kicad/digital_probe/digital_probe.sch-bak
Connections:
- D2 pad 2: GND -> +3V3
Routing:
- net +3V3: track 42.2 -> 42.7 mm
