File: kicad/digital_probe/digital_probe.kicad_pcb (KiCad board)
At the start: 2 copper layers, 45.5 x 72.4 mm, 33 parts, among them J1 Conn_02x08_Odd_Even, J2 Conn_02x08_Odd_Even, J3 Conn_02x25_Odd_Even, J4 D8-15 Vref, J5 D0-7 Vref, U1 MC33375ST

Commit message: изменено:      kicad/digital_probe/digital_probe.kicad_pcb 	изменено:      kicad/digital_probe/digital_probe.kicad_pcb-bak 	новый файл:    kicad/digital_probe/gerber/digital_probe.zip
Parts:
- moved C2 0.11 mm to (55.1, 92.2)
- moved C5 0.10 mm to (55.1, 99.1)
- moved C6 0.05 mm to (55.1, 96.9)
- moved C3 0.05 mm to (55.1, 94.3)
Routing:
- net Net-(D2-Pad6): track 19.8 -> 20.9 mm
- net Net-(D2-Pad7): track 22.0 -> 23.1 mm
- net GND: vias 4 -> 6
Other:
- outline, holes or cut-outs redrawn
