File: kicad/digital_probe/digital_probe.sch (KiCad schematic (older format))
At the start: 33 parts, among them J1 Conn_02x08_Odd_Even, J2 Conn_02x08_Odd_Even, J3 Conn_02x25_Odd_Even, J4 D8-15 Vref, J5 D0-7 Vref, U1 MC33375ST

Commit message: изменено:      kicad/digital_probe/digital_probe-cache.lib 	изменено:      kicad/digital_probe/digital_probe.kicad_pcb 	изменено:      kicad/digital_probe/digital_probe.kicad_pcb-bak 	изменено:      kicad/digital_probe/digital_probe.sch 	изменено:      kicad/digital_probe/digital_probe.sch-bak
Parts:
- D2: symbol My_Library:SN65LVDS1677 -> digital_probe-rescue:SN65LVDS1677-My_Library
- J4, J5: symbol My_Library:Conn -> digital_probe-rescue:Conn-My_Library
- U1: symbol My_Library:MC33375ST -> digital_probe-rescue:MC33375ST-My_Library
Connections:
- net GND: no longer D2.2 (Vcc)
Changed lines of the file:
@@
 $EndDescr
 $Comp
-L My_Library:SN65LVDS1677 D2
+L digital_probe-rescue:SN65LVDS1677-My_Library D2
 U 1 1 62978B70
 P 3500 2850
@@
 $EndComp
 $Comp
-L My_Library:SN65LVDS1677 D2
+L digital_probe-rescue:SN65LVDS1677-My_Library D2
 U 2 1 62979ACA
 P 3500 4450
@@
 $EndComp
 $Comp
-L My_Library:SN65LVDS1677 D2
+L digital_probe-rescue:SN65LVDS1677-My_Library D2
 U 3 1 6297C4AE
 P 3500 5950
@@
 $EndComp
 $Comp
-L My_Library:SN65LVDS1677 D2
+L digital_probe-rescue:SN65LVDS1677-My_Library D2
 U 4 1 6297D457
 P 3500 7450
@@
 Connection ~ 3650 3450
 $Comp
-L My_Library:MC33375ST U1
+L digital_probe-rescue:MC33375ST-My_Library U1
 U 1 1 62BE7183
 P 5200 4200
@@
 D15
 $Comp
-L My_Library:Conn J4
+L digital_probe-rescue:Conn-My_Library J4
 U 1 1 631BF0C8
 P 4850 5100
@@
 $EndComp
 $Comp
-L My_Library:Conn J5
+L digital_probe-rescue:Conn-My_Library J5
 U 1 1 631C23C8
 P 5550 5100

Commit message: изменено:      kicad/digital_probe/digital_probe-cache.lib 	изменено:      kicad/digital_probe/digital_probe.kicad_pcb 	изменено:      kicad/digital_probe/digital_probe.kicad_pcb-bak 	изменено:      kicad/digital_probe/digital_probe.sch 	изменено:      kicad/digital_probe/digital_probe.sch-bak
Changed lines of the file:
@@
 Connection ~ 3450 3450
 Connection ~ 3550 3450
-Wire Wire Line
-	3550 3450 3650 3450
 $Comp
 L Device:R R15
@@
 	1    0    0    -1
 $EndComp
-Wire Wire Line
-	3650 3450 3750 3450
-Connection ~ 3650 3450
 $Comp
 L digital_probe-rescue:MC33375ST-My_Library U1
@@
 Text Label 5550 5300 0    50   ~ 0
 +4v
+Wire Wire Line
+	3550 3450 3750 3450
 $EndSCHEMATC

Commit message: новый файл:    Documents/IMG_20221001_132513.jpg 	изменено:      kicad/digital_probe/digital_probe-cache.lib 	изменено:      kicad/digital_probe/digital_probe.kicad_pcb 	изменено:      kicad/digital_probe/digital_probe.kicad_pcb-bak 	изменено:      kicad/digital_probe/digital_probe.sch 	изменено:      kicad/digital_probe/digital_probe.sch-bak
Parts:
- D2: symbol digital_probe-rescue:SN65LVDS1677-My_Library -> digital_probe-rescue:SN65LVDS1677-My_Library-digital_probe-rescue
- J4, J5: symbol digital_probe-rescue:Conn-My_Library -> digital_probe-rescue:Conn-My_Library-digital_probe-rescue
- U1: symbol digital_probe-rescue:MC33375ST-My_Library -> digital_probe-rescue:MC33375ST-My_Library-digital_probe-rescue
Changed lines of the file:
@@
 $EndDescr
 $Comp
-L digital_probe-rescue:SN65LVDS1677-My_Library D2
+L digital_probe-rescue:SN65LVDS1677-My_Library-digital_probe-rescue D2
 U 1 1 62978B70
 P 3500 2850
@@
 $EndComp
 $Comp
-L digital_probe-rescue:SN65LVDS1677-My_Library D2
+L digital_probe-rescue:SN65LVDS1677-My_Library-digital_probe-rescue D2
 U 2 1 62979ACA
 P 3500 4450
@@
 $EndComp
 $Comp
-L digital_probe-rescue:SN65LVDS1677-My_Library D2
+L digital_probe-rescue:SN65LVDS1677-My_Library-digital_probe-rescue D2
 U 3 1 6297C4AE
 P 3500 5950
@@
 $EndComp
 $Comp
-L digital_probe-rescue:SN65LVDS1677-My_Library D2
+L digital_probe-rescue:SN65LVDS1677-My_Library-digital_probe-rescue D2
 U 4 1 6297D457
 P 3500 7450
@@
 $EndComp
 $Comp
-L digital_probe-rescue:MC33375ST-My_Library U1
+L digital_probe-rescue:MC33375ST-My_Library-digital_probe-rescue U1
 U 1 1 62BE7183
 P 5200 4200
@@
 D15
 $Comp
-L digital_probe-rescue:Conn-My_Library J4
+L digital_probe-rescue:Conn-My_Library-digital_probe-rescue J4
 U 1 1 631BF0C8
 P 4850 5100
@@
 $EndComp
 $Comp
-L digital_probe-rescue:Conn-My_Library J5
+L digital_probe-rescue:Conn-My_Library-digital_probe-rescue J5
 U 1 1 631C23C8
 P 5550 5100
